File: 001 PCB/KICAD/COPPER KICAD/TheENDGAME2024_COPPER.kicad_sch (KiCad schematic)
At the start: 74 parts, among them SW10 SW_Push, SW11 SW_Push, SW12 SW_Push, SW13 SW_Push, SW14 SW_Push, SW15 SW_Push, SW16 SW_Push, SW17 SW_Push, SW18 SW_Push, SW19 SW_Push, SW2 SW_Push, SW20 SW_Push, SW21 SW_Push, SW22 SW_Push, SW23 SW_Push, SW24 SW_Push, SW25 SW_Push, SW26 SW_Push, SW27 SW_Push, SW28 SW_Push, SW29 SW_Push, SW3 SW_Push, SW30 SW_Push, SW31 SW_Push, SW32 SW_Push, SW33 SW_Push, SW34 SW_Push, SW35 SW_Push, SW36 SW_Push, SW37 SW_Push, SW4 SW_Push, SW5 SW_Push, SW6 SW_Push, SW7 SW_Push, SW8 SW_Push, SW9 SW_Push, U2 RP2040-Zero_stolen_from_Purox

Commit message: Add Choc V1/V2 hot-swap support and JLCPCB fabrication package
Parts:
- SW10, SW11, SW12, SW13, SW14, SW15, SW16, SW17, SW18, SW2, SW20, SW21, SW22, SW24, SW25, SW26, SW27, SW28, SW29, SW3, SW30, SW31, SW32, SW33, SW34, SW35, SW36, SW4, SW6, SW7, SW8, SW9: footprint TheEndgame2024:SW_choc_v1_HSxSolder_1u_filets_MBK_blk fixxed flipped solder pads -> TheEndgame2024:SW_choc_v1_v2_HS_1u
- SW19, SW23, SW37, SW5: footprint TheEndgame2024:SW_choc_v1_HSxSolder_1.5u_filets_MBK_blk fixxed flipped solder pads -> TheEndgame2024:SW_choc_v1_v2_HS_1.5u
Changed lines of the file:
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@@
 			)
 		)
-		(property "Footprint" "TheEndgame2024:SW_choc_v1_HSxSolder_1u_filets_MBK_blk fixxed flipped solder pads"
+		(property "Footprint" "TheEndgame2024:SW_choc_v1_v2_HS_1u"
 			(at 156.21 35.56 0)
 			(effects
@@
 			)
 		)
-		(property "Footprint" "TheEndgame2024:SW_choc_v1_HSxSolder_1.5u_filets_MBK_blk fixxed flipped solder pads"
+		(property "Footprint" "TheEndgame2024:SW_choc_v1_v2_HS_1.5u"
 			(at 142.24 90.17 0)
 			(effects
@@
 			)
 		)
-		(property "Footprint" "TheEndgame2024:SW_choc_v1_HSxSolder_1u_filets_MBK_blk fixxed flipped solder pads"
+		(property "Footprint" "TheEndgame2024:SW_choc_v1_v2_HS_1u"
 			(at 226.06 35.56 0)
 			(effects
@@
 			)
 		)
-		(property "Footprint" "TheEndgame2024:SW_choc_v1_HSxSolder_1u_filets_MBK_blk fixxed flipped solder pads"
+		(property "Footprint" "TheEndgame2024:SW_choc_v1_v2_HS_1u"
 			(at 184.15 72.39 0)
 			(effects
@@
 			)
 		)
-		(property "Footprint" "TheEndgame2024:SW_choc_v1_HSxSolder_1u_filets_MBK_blk fixxed flipped solder pads"
+		(property "Footprint" "TheEndgame2024:SW_choc_v1_v2_HS_1u"
 			(at 198.12 72.39 0)
 			(effects
@@
 			)
 		)
-		(property "Footprint" "TheEndgame2024:SW_choc_v1_HSxSolder_1u_filets_MBK_blk fixxed flipped solder pads"
+		(property "Footprint" "TheEndgame2024:SW_choc_v1_v2_HS_1u"
 			(at 156.21 53.34 0)
 			(effects
@@
 			)
 		)
-		(property "Footprint" "TheEndgame2024:SW_choc_v1_HSxSolder_1u_filets_MBK_blk fixxed flipped solder pads"
+		(property "Footprint" "TheEndgame2024:SW_choc_v1_v2_HS_1u"
 			(at 198.12 35.56 0)
 			(effects
@@
 			)
 		)
-		(property "Footprint" "TheEndgame2024:SW_choc_v1_HSxSolder_1u_filets_MBK_blk fixxed flipped solder pads"
+		(property "Footprint" "TheEndgame2024:SW_choc_v1_v2_HS_1u"
 			(at 170.18 53.34 0)
 			(effects
@@
 			)
 		)
-		(property "Footprint" "TheEndgame2024:SW_choc_v1_HSxSolder_1u_filets_MBK_blk fixxed flipped solder pads"
+		(property "Footprint" "TheEndgame2024:SW_choc_v1_v2_HS_1u"
 			(at 254 35.56 0)
 			(effects
@@
 			)
 		)
-		(property "Footprint" "TheEndgame2024:SW_choc_v1_HSxSolder_1.5u_filets_MBK_blk fixxed flipped solder pads"
+		(property "Footprint" "TheEndgame2024:SW_choc_v1_v2_HS_1.5u"
 			(at 198.12 90.17 0)
 			(effects
@@
 			)
 		)
-		(property "Footprint" "TheEndgame2024:SW_choc_v1_HSxSolder_1u_filets_MBK_blk fixxed flipped solder pads"
+		(property "Footprint" "TheEndgame2024:SW_choc_v1_v2_HS_1u"
 			(at 184.15 90.17 0)
 			(effects
@@
 			)
 		)
-		(property "Footprint" "TheEndgame2024:SW_choc_v1_HSxSolder_1u_filets_MBK_blk fixxed flipped solder pads"
+		(property "Footprint" "TheEndgame2024:SW_choc_v1_v2_HS_1u"
 			(at 254 72.39 0)
 			(effects
@@
 			)
 		)
-		(property "Footprint" "TheEndgame2024:SW_choc_v1_HSxSolder_1u_filets_MBK_blk fixxed flipped solder pads"
+		(property "Footprint" "TheEndgame2024:SW_choc_v1_v2_HS_1u"
 			(at 170.18 72.39 0)
 			(effects
@@
 			)
 		)
-		(property "Footprint" "TheEndgame2024:SW_choc_v1_HSxSolder_1u_filets_MBK_blk fixxed flipped solder pads"
+		(property "Footprint" "TheEndgame2024:SW_choc_v1_v2_HS_1u"
 			(at 240.03 35.56 0)
 			(effects
@@
 			)
 		)
-		(property "Footprint" "TheEndgame2024:SW_choc_v1_HSxSolder_1u_filets_MBK_blk fixxed flipped solder pads"
+		(property "Footprint" "TheEndgame2024:SW_choc_v1_v2_HS_1u"
 			(at 184.15 35.56 0)
 			(effects
@@
 			)
 		)
-		(property "Footprint" "TheEndgame2024:SW_choc_v1_HSxSolder_1u_filets_MBK_blk fixxed flipped solder pads"
+		(property "Footprint" "TheEndgame2024:SW_choc_v1_v2_HS_1u"
 			(at 142.24 35.56 0)
 			(effects
@@
 			)
 		)
-		(property "Footprint" "TheEndgame2024:SW_choc_v1_HSxSolder_1.5u_filets_MBK_blk fixxed flipped solder pads"
+		(property "Footprint" "TheEndgame2024:SW_choc_v1_v2_HS_1.5u"
 			(at 212.09 90.17 0)
 			(effects
@@
 			)
 		)
-		(property "Footprint" "TheEndgame2024:SW_choc_v1_HSxSolder_1u_filets_MBK_blk fixxed flipped solder pads"
+		(property "Footprint" "TheEndgame2024:SW_choc_v1_v2_HS_1u"
 			(at 212.09 53.34 0)
 			(effects
@@
 			)
 		)
-		(property "Footprint" "TheEndgame2024:SW_choc_v1_HSxSolder_1u_filets_MBK_blk fixxed flipped solder pads"
+		(property "Footprint" "TheEndgame2024:SW_choc_v1_v2_HS_1u"
 			(at 240.03 72.39 0)
 			(effects
@@
 			)
 		)
-		(property "Footprint" "TheEndgame2024:SW_choc_v1_HSxSolder_1.5u_filets_MBK_blk fixxed flipped solder pads"
+		(property "Footprint" "TheEndgame2024:SW_choc_v1_v2_HS_1.5u"
 			(at 267.97 90.17 0)
 			(effects
@@
 			)
 		)
-		(property "Footprint" "TheEndgame2024:SW_choc_v1_HSxSolder_1u_filets_MBK_blk fixxed flipped solder pads"
+		(property "Footprint" "TheEndgame2024:SW_choc_v1_v2_HS_1u"
 			(at 198.12 53.34 0)
 			(effects
@@
 			)
 		)
-		(property "Footprint" "TheEndgame2024:SW_choc_v1_HSxSolder_1u_filets_MBK_blk fixxed flipped solder pads"
+		(property "Footprint" "TheEndgame2024:SW_choc_v1_v2_HS_1u"
 			(at 184.15 53.34 0)
 			(effects
@@
 			)
 		)
-		(property "Footprint" "TheEndgame2024:SW_choc_v1_HSxSolder_1u_filets_MBK_blk fixxed flipped solder pads"
+		(property "Footprint" "TheEndgame2024:SW_choc_v1_v2_HS_1u"
 			(at 226.06 72.39 0)
 			(effects
@@
 			)
 		)
-		(property "Footprint" "TheEndgame2024:SW_choc_v1_HSxSolder_1u_filets_MBK_blk fixxed flipped solder pads"
+		(property "Footprint" "TheEndgame2024:SW_choc_v1_v2_HS_1u"
 			(at 240.03 53.34 0)
 			(effects
@@
 			)
 		)
-		(property "Footprint" "TheEndgame2024:SW_choc_v1_HSxSolder_1u_filets_MBK_blk fixxed flipped solder pads"
+		(property "Footprint" "TheEndgame2024:SW_choc_v1_v2_HS_1u"
 			(at 156.21 72.39 0)
 			(effects
@@
 			)
 		)
-		(property "Footprint" "TheEndgame2024:SW_choc_v1_HSxSolder_1u_filets_MBK_blk fixxed flipped solder pads"
+		(property "Footprint" "TheEndgame2024:SW_choc_v1_v2_HS_1u"
 			(at 267.97 72.39 0)
 			(effects
@@
 			)
 		)
-		(property "Footprint" "TheEndgame2024:SW_choc_v1_HSxSolder_1u_filets_MBK_blk fixxed flipped solder pads"
+		(property "Footprint" "TheEndgame2024:SW_choc_v1_v2_HS_1u"
 			(at 212.09 35.56 0)
 			(effects
@@
 			)
 		)
-		(property "Footprint" "TheEndgame2024:SW_choc_v1_HSxSolder_1u_filets_MBK_blk fixxed flipped solder pads"
+		(property "Footprint" "TheEndgame2024:SW_choc_v1_v2_HS_1u"
 			(at 254 53.34 0)
 			(effects
@@
 			)
 		)
-		(property "Footprint" "TheEndgame2024:SW_choc_v1_HSxSolder_1u_filets_MBK_blk fixxed flipped solder pads"
+		(property "Footprint" "TheEndgame2024:SW_choc_v1_v2_HS_1u"
 			(at 212.09 72.39 0)
 			(effects
@@
 			)
 		)
-		(property "Footprint" "TheEndgame2024:SW_choc_v1_HSxSolder_1u_filets_MBK_blk fixxed flipped solder pads"
+		(property "Footprint" "TheEndgame2024:SW_choc_v1_v2_HS_1u"
 			(at 170.18 35.56 0)
 			(effects
@@
 			)
 		)
-		(property "Footprint" "TheEndgame2024:SW_choc_v1_HSxSolder_1u_filets_MBK_blk fixxed flipped solder pads"
+		(property "Footprint" "TheEndgame2024:SW_choc_v1_v2_HS_1u"
 			(at 226.06 53.34 0)
 			(effects
@@
 			)
 		)
-		(property "Footprint" "TheEndgame2024:SW_choc_v1_HSxSolder_1u_filets_MBK_blk fixxed flipped solder pads"
+		(property "Footprint" "TheEndgame2024:SW_choc_v1_v2_HS_1u"
 			(at 267.97 35.56 0)
 			(effects
@@
 			)
 		)
-		(property "Footprint" "TheEndgame2024:SW_choc_v1_HSxSolder_1u_filets_MBK_blk fixxed flipped solder pads"
+		(property "Footprint" "TheEndgame2024:SW_choc_v1_v2_HS_1u"
 			(at 142.24 53.34 0)
 			(effects
@@
 			)
 		)
-		(property "Footprint" "TheEndgame2024:SW_choc_v1_HSxSolder_1u_filets_MBK_blk fixxed flipped solder pads"
+		(property "Footprint" "TheEndgame2024:SW_choc_v1_v2_HS_1u"
 			(at 267.97 53.34 0)
 			(effects
@@
 			)
 		)
-		(property "Footprint" "TheEndgame2024:SW_choc_v1_HSxSolder_1u_filets_MBK_blk fixxed flipped solder pads"
+		(property "Footprint" "TheEndgame2024:SW_choc_v1_v2_HS_1u"
 			(at 142.24 72.39 0)
 			(effects
@@
 			)
 		)
-		(property "Footprint" "TheEndgame2024:SW_choc_v1_HSxSolder_1u_filets_MBK_blk fixxed flipped solder pads"
+		(property "Footprint" "TheEndgame2024:SW_choc_v1_v2_HS_1u"
 			(at 226.06 90.17 0)
 			(effects
