File: 001 PCB/KICAD/NICE NANO WIRELESS/TheEndgame2024_NiceNano.kicad_sch (KiCad schematic)
At the start: 79 parts, among them J1 BATTERY_WIRES, SW10 SW_Push, SW11 SW_Push, SW12 SW_Push, SW13 SW_Push, SW14 SW_Push, SW15 SW_Push, SW16 SW_Push, SW17 SW_Push, SW18 SW_Push, SW19 SW_Push, SW2 SW_Push, SW20 SW_Push, SW21 SW_Push, SW22 SW_Push, SW23 SW_Push, SW24 SW_Push, SW25 SW_Push, SW26 SW_Push, SW27 SW_Push, SW28 SW_Push, SW29 SW_Push, SW3 SW_Push, SW30 SW_Push, SW31 SW_Push, SW32 SW_Push, SW33 SW_Push, SW34 SW_Push, SW35 SW_Push, SW36 SW_Push, SW37 SW_Push, SW38 PCM12SMTR, SW4 SW_Push, SW5 SW_Push, SW6 SW_Push, SW7 SW_Push, SW8 SW_Push, SW9 SW_Push, U2 nice!nano_v2

Commit message: Widen key halves for controller clearance and add axial resistors
Parts:
- R1, R2: footprint Resistor_SMD:R_0603_1608Metric -> NanoWireless:R_Axial_DIN0207_L6.3mm_D2.5mm_P10.16mm_Horizontal
Changed lines of the file:
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@@
 (global_label "gnd" (shape passive) (at 213.3600 143.5100 180) (effects (font (size 1.27 1.27)) (justify right)) (property "Intersheetrefs" "${INTERSHEET_REFS}" (at 213.3600 143.5100 0) (effects (font (size 1.27 1.27)) (hide yes))))
 (symbol (lib_id "Device:R") (at 148.5900 139.7000 0) (unit 1) (in_bom yes) (on_board yes) (dnp no)
- (property "Reference" "R1" (at 154.9400 138.4300 0) (effects (font (size 1.27 1.27)))) (property "Value" "330" (at 154.9400 140.9700 0) (effects (font (size 1.27 1.27)))) (property "Footprint" "Resistor_SMD:R_0603_1608Metric" (at 148.5900 139.7000 0) (effects (font (size 1.27 1.27)) (hide yes))) (property "Datasheet" "" (at 148.5900 139.7000 0) (effects (font (size 1.27 1.27)) (hide yes)))
+ (property "Reference" "R1" (at 154.9400 138.4300 0) (effects (font (size 1.27 1.27)))) (property "Value" "330" (at 154.9400 140.9700 0) (effects (font (size 1.27 1.27)))) (property "Footprint" "NanoWireless:R_Axial_DIN0207_L6.3mm_D2.5mm_P10.16mm_Horizontal" (at 148.5900 139.7000 0) (effects (font (size 1.27 1.27)) (hide yes))) (property "Datasheet" "" (at 148.5900 139.7000 0) (effects (font (size 1.27 1.27)) (hide yes)))
  (pin "1")
 (pin "2")
@@
 (global_label "LED_DIN" (shape passive) (at 148.5900 143.5100 180) (effects (font (size 1.27 1.27)) (justify right)) (property "Intersheetrefs" "${INTERSHEET_REFS}" (at 148.5900 143.5100 0) (effects (font (size 1.27 1.27)) (hide yes))))
 (symbol (lib_id "Device:R") (at 148.5900 166.3700 0) (unit 1) (in_bom yes) (on_board yes) (dnp no)
- (property "Reference" "R2" (at 154.9400 165.1000 0) (effects (font (size 1.27 1.27)))) (property "Value" "100k" (at 154.9400 167.6400 0) (effects (font (size 1.27 1.27)))) (property "Footprint" "Resistor_SMD:R_0603_1608Metric" (at 148.5900 166.3700 0) (effects (font (size 1.27 1.27)) (hide yes))) (property "Datasheet" "" (at 148.5900 166.3700 0) (effects (font (size 1.27 1.27)) (hide yes)))
+ (property "Reference" "R2" (at 154.9400 165.1000 0) (effects (font (size 1.27 1.27)))) (property "Value" "100k" (at 154.9400 167.6400 0) (effects (font (size 1.27 1.27)))) (property "Footprint" "NanoWireless:R_Axial_DIN0207_L6.3mm_D2.5mm_P10.16mm_Horizontal" (at 148.5900 166.3700 0) (effects (font (size 1.27 1.27)) (hide yes))) (property "Datasheet" "" (at 148.5900 166.3700 0) (effects (font (size 1.27 1.27)) (hide yes)))
  (pin "1")
 (pin "2")
