File: 001 PCB/KICAD/NICE NANO CIRQUE/TheEndgame2024_NiceNanoCirque.kicad_pcb (KiCad board)
At the start: 2 copper layers, 239 x 96.1 mm, 99 parts, among them J1 BATTERY_WIRES, J2 Cirque FFC 12P 0.5mm, SW10 SW_Push, SW11 SW_Push, SW12 SW_Push, SW13 SW_Push, SW14 SW_Push, SW15 SW_Push, SW16 SW_Push, SW17 SW_Push, SW18 SW_Push, SW19 SW_Push, SW2 SW_Push, SW20 SW_Push, SW21 SW_Push, SW22 SW_Push, SW23 SW_Push, SW24 SW_Push, SW25 SW_Push, SW26 SW_Push, SW27 SW_Push, SW28 SW_Push, SW29 SW_Push, SW3 SW_Push, SW30 SW_Push, SW31 SW_Push, SW32 SW_Push, SW33 SW_Push, SW34 SW_Push, SW35 SW_Push, SW36 SW_Push, SW37 SW_Push, SW38 PCM12SMTR, SW4 SW_Push, SW5 SW_Push, SW6 SW_Push, SW7 SW_Push, SW8 SW_Push, SW9 SW_Push, U2 nice!nano_v2

Commit message: Recess the Cirque power switch and add photo silkscreen artwork
Move SW38 so its slider stays 0.46 mm inside the PCB edge, re-route and
update the case check. Add a dithered photo (0.25 mm dots) to both
silkscreen layers, mirrored on the underside, kept clear of edges and the
mounting-hole ring art; DRC has 0 errors. Router now ignores a net's own
drill holes.

Co-Authored-By: Claude Opus 5.5 <noreply@anthropic.com>
Parts:
- moved SW38 1.80 mm to (150.0, 66.3)
Routing:
- net VBAT: track 93.8 -> 92.0 mm
- net VBAT_SW: track 10.8 -> 11.4 mm
