File: 001 PCB/KICAD/NICE NANO CIRQUE/TheEndgame2024_NiceNanoCirque.kicad_pcb (KiCad board)
At the start: 2 copper layers, 239 x 96.1 mm, 99 parts, among them J1 BATTERY_WIRES, J2 Cirque FFC 12P 0.5mm, SW10 SW_Push, SW11 SW_Push, SW12 SW_Push, SW13 SW_Push, SW14 SW_Push, SW15 SW_Push, SW16 SW_Push, SW17 SW_Push, SW18 SW_Push, SW19 SW_Push, SW2 SW_Push, SW20 SW_Push, SW21 SW_Push, SW22 SW_Push, SW23 SW_Push, SW24 SW_Push, SW25 SW_Push, SW26 SW_Push, SW27 SW_Push, SW28 SW_Push, SW29 SW_Push, SW3 SW_Push, SW30 SW_Push, SW31 SW_Push, SW32 SW_Push, SW33 SW_Push, SW34 SW_Push, SW35 SW_Push, SW36 SW_Push, SW37 SW_Push, SW38 PCM12SMTR, SW4 SW_Push, SW5 SW_Push, SW6 SW_Push, SW7 SW_Push, SW8 SW_Push, SW9 SW_Push, U2 nice!nano_v2

Commit message: Fix second pre-order review findings on the Cirque build
Board:
- Extend the FFC notch to PCB X 168.9 (Y 117-129) to match where
  Cirque's drawing and photo put the pad connector (12.5-18.4 mm out,
  slot at 15.7-16.4 mm), and move J2 to X 176.0 so the cable has ~4 mm
  for its bend. Pins 1/3 and the ground via fan out under J2's body
  because SW22's socket pad sits 1 mm past the pad row.
- Store the 0.2 mm copper-to-edge rule in the project file. The Gerber
  export refills zones with the project rules, so the shipped pour had
  run right up to the board edge.
- Keep router vias 0.3 mm from every solder pad (two had landed in R4
  and R1 pads).
- Keep the underside photo 0.2 mm from pad openings, holes, vias and
  part outlines, leave J2 blank, and drop the off-board 300 x 200 mm
  silkscreen frame.
- No stencil paste on the hand-soldered sockets and SW38.
- Repeatable schematic UUIDs.
- New tools/verify_cirque_gerbers.py checks the exported ZIP: copper to
  edge, paste over holes, silkscreen in openings and slivers.

Case:
- Pad connector proxy at its real position, with computed notch-fit
  checks and J2/FFC proxies.
- Carrier ring widened to 0.2 mm inside the counterbore so it is
  centred, kept on board material, and printed 0.2 mm short for a foam
  shim.
- LED pocket widened to cover the LED's pads; SW38 proxies corrected.
- The LED-logo light chamber keeps a 0.5 mm wall to the grommet recess.
- Layout sketch, docs and validation reports updated.

Co-Authored-By: Claude Opus 5.5 <noreply@anthropic.com>
Parts:
- moved J2 2.70 mm to (176.0, 123.0)
Routing:
- net VCC_SW: track 151.5 -> 157.9 mm, vias 6 -> 9
- net gnd: track 43.5 -> 39.4 mm, vias 9 -> 7
- net SDA: track 52.2 -> 48.1 mm
- net SCL: track 40.9 -> 43.8 mm
- net DR: track 35.6 -> 36.7 mm
- net LED_DATA: track 129.0 -> 130.0 mm
Other:
- outline, holes or cut-outs redrawn
