File: 001 PCB/KICAD/NICE NANO CIRQUE/TheEndgame2024_NiceNanoCirque.kicad_sch (KiCad schematic)
At the start: 83 parts, among them J1 BATTERY_WIRES, J2 Cirque FFC 12P 0.5mm, SW10 SW_Push, SW11 SW_Push, SW12 SW_Push, SW13 SW_Push, SW14 SW_Push, SW15 SW_Push, SW16 SW_Push, SW17 SW_Push, SW18 SW_Push, SW19 SW_Push, SW2 SW_Push, SW20 SW_Push, SW21 SW_Push, SW22 SW_Push, SW23 SW_Push, SW24 SW_Push, SW25 SW_Push, SW26 SW_Push, SW27 SW_Push, SW28 SW_Push, SW29 SW_Push, SW3 SW_Push, SW30 SW_Push, SW31 SW_Push, SW32 SW_Push, SW33 SW_Push, SW34 SW_Push, SW35 SW_Push, SW36 SW_Push, SW37 SW_Push, SW38 PCM12SMTR, SW4 SW_Push, SW5 SW_Push, SW6 SW_Push, SW7 SW_Push, SW8 SW_Push, SW9 SW_Push, U2 nice!nano_v2

Commit message: Fix pre-order review findings on the nice!nano + Cirque build
- Reverse J2's pin order: the FFC keeps conductor order through its bend,
  so pad pin N lands on J2 pin 13-N (DR 9, SCL 4, SDA 3, GND 2, VDD 1).
- Move J2 3.7 mm from the notch so the cable can bend; widen the notch;
  correct the AFC01 footprint (nails at +-4.45, 5.75 mm body courtyard);
  re-join the row traces it displaced.
- Keep copper 0.2 mm from edges and 0.25 mm from holes (refilled pour).
- Re-cut the case's front pocket to the real PCB outline (the front tabs
  overlapped the case wall by 0.48 mm) and check 0.3 mm clearance.
- Keep the underside photo exactly 0.4 mm from edges.
- Add paste layers to the Gerber ZIP and the 36 1N4148W diodes to the
  JLCPCB BOM/CPL; document cable type, length and checks.

DRC: 0 errors, 0 unconnected, 0 parity issues; ERC clean.

Co-Authored-By: Claude Opus 5.5 <noreply@anthropic.com>
Parts:
- D10, D11, D12, D13, D14, D15, D17, D18, D19, D20, D22, D23, D24, D25, D26, D27, D28, D29, D32, D33, D34, D35, D36, D37, D38, D39, D40, D41, D44, D45, D46, D47, D5, D6, D7, D8: value D_Small -> 1N4148W; LCSC (none) -> C81598
Connections:
- net DR: now also J2.9 (Pin_9); no longer J2.4 (Pin_4)
- net SCL: now also J2.4 (Pin_4); no longer J2.9 (Pin_9)
- net SDA: now also J2.3 (Pin_3); no longer J2.10 (Pin_10)
- net VCC_SW: now also J2.1 (Pin_1); no longer J2.12 (Pin_12)
- net gnd: now also J2.2 (Pin_2); no longer J2.11 (Pin_11)
Other:
- note added: "Cirque TM040040 (Pinnacle) in I2C mode: remove R1 on the pad module. Pad pins 4 DR, 9 SCL, 10 SDA, 11 GND, 12 VDD arrive on J2 pins 9, 4, 3, 2, 1 (the FFC path reverses the order; pad pin N = J2 pin 13-N)."
- note removed: "Cirque TM040040 (Pinnacle) in I2C mode: remove R1 on the pad module. FFC pins: 4 DR, 9 SCL, 10 SDA, 11 GND, 12 VDD 3.3 V."
